File: tools/GS/GS.kicad_pcb (KiCad board)
At the start: 2 copper layers, 25 x 57.5 mm, 22 parts, among them CN1 USB-B-MICRO, J1 SMA, SW1 RST, SW2 PRG, U1 L78L05_SOT89, U2 TWE_LITE_SMD, U3 FT231XQ

Commit message: Update GS
Routing:
- net Net-(C6-Pad1): track 13.4 -> 12.7 mm
Changed lines of the file:
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@@
     (thickness 1.6)
     (drawings 18)
-    (tracks 193)
+    (tracks 195)
     (zones 0)
     (modules 22)
@@
     (pad_to_mask_clearance 0)
     (aux_axis_origin 0 0)
-    (visible_elements FFFFFF7F)
+    (visible_elements 7FFFFFFF)
     (pcbplotparams
-      (layerselection 0x010fc_ffffffff)
-      (usegerberextensions false)
+      (layerselection 0x010f0_ffffffff)
+      (usegerberextensions true)
       (usegerberattributes false)
       (usegerberadvancedattributes false)
@@
       (outputformat 1)
       (mirror false)
-      (drillshape 1)
+      (drillshape 0)
       (scaleselection 1)
-      (outputdirectory ""))
+      (outputdirectory "Gerber"))
   )
   (net 0 "")
@@
   (gr_line (start 60 80) (end 65.5 80) (layer Edge.Cuts) (width 0.15))
   (gr_line (start 57.5 25) (end 57.5 77.5) (layer Edge.Cuts) (width 0.15))
-  (via (at 65 65) (size 0.6) (drill 0.3) (layers F.Cu B.Cu) (net 20))
   (via (at 66.5 61) (size 0.6) (drill 0.3) (layers F.Cu B.Cu) (net 2))
   (segment (start 66 63.0625) (end 66 61.5) (width 0.25) (layer F.Cu) (net 2))
@@
   (segment (start 65.5 52.29) (end 65.555 52.235) (width 0.25) (layer F.Cu) (net 9))
   (segment (start 65.5 54) (end 65.5 52.29) (width 0.25) (layer F.Cu) (net 9))
+  (via (at 65 65) (size 0.6) (drill 0.3) (layers F.Cu B.Cu) (net 20))
   (segment (start 73.2427 65) (end 75.9097 65) (width 0.25) (layer F.Cu) (net 20))
   (segment (start 74.5 65) (end 75.9097 65) (width 0.25) (layer F.Cu) (net 20))
@@
   (segment (start 65 70) (end 65 66.9375) (width 0.25) (layer F.Cu) (net 31))
   (segment (start 64.5 70.5) (end 65 70) (width 0.25) (layer F.Cu) (net 31))
-  (segment (start 64.5 72) (end 64.5 70.5) (width 0.25) (layer F.Cu) (net 31))
-  (segment (start 65.5 73) (end 64.5 72) (width 0.25) (layer F.Cu) (net 31))
-  (segment (start 69.75 73) (end 65.5 73) (width 0.25) (layer F.Cu) (net 31))
-  (segment (start 70 75.325) (end 70 73.25) (width 0.25) (layer F.Cu) (net 31))
-  (segment (start 70 73.25) (end 69.75 73) (width 0.25) (layer F.Cu) (net 31))
+  (segment (start 70 73.25) (end 70 75.325) (width 0.25) (layer F.Cu) (net 31))
+  (segment (start 66.03859 71.175) (end 67.3136 72.45001) (width 0.25) (layer F.Cu) (net 31))
+  (segment (start 67.3136 72.45001) (end 69.20001 72.45001) (width 0.25) (layer F.Cu) (net 31))
+  (segment (start 69.20001 72.45001) (end 70 73.25) (width 0.25) (layer F.Cu) (net 31))
+  (segment (start 65.375 71.175) (end 65 70.8) (width 0.25) (layer F.Cu) (net 31))
+  (segment (start 66.03859 71.175) (end 65.375 71.175) (width 0.25) (layer F.Cu) (net 31))
+  (segment (start 65 70) (end 65 70.8) (width 0.25) (layer F.Cu) (net 31))
   (segment (start 60.5 27.875) (end 60.5 30.125) (width 0.25) (layer F.Cu) (net 38))
   (segment (start 62.5 30.125) (end 62.5 27.875) (width 0.25) (layer F.Cu) (net 39))
