File: PCB/CanSat2020_P/CanSat2020_P.kicad_pcb (KiCad board)
At the start: 2 copper layers, 4.3 x 3.1 mm, 82 parts, among them J1 GNSS Antenna, J2 Debug_L0, J3 Debug_F2, M1 Motor_L, M2 Motor_R, P1 C1098, Q1 FDS4935A, Q2 MTM231102LBF, Q3 2SC2712, SW1 POWER, U1 STM32L081CBTx, U10 BD6231F, U12 BD6231F, U2 STM32F205RFTx, U3 INA226, U4 TPS62162DSG, U5 W25Q128JVE, U6 LSM303A, U7 ADXL375, U8 L76, U9 VL53L0X

Commit message: Update PCB
Parts:
- added C21: 0.1u, Capacitor_SMD:C_0603_1608Metric_Pad1.05x0.95mm_HandSolder, F.Cu at (107.4, 72.9)
- added C22: 0.1u, Capacitor_SMD:C_0603_1608Metric_Pad1.05x0.95mm_HandSolder, F.Cu at (105.4, 72.9)
- added P2: Charge, Connector_JST:JST_EH_B03B-EH-A_1x03_P2.50mm_Vertical, B.Cu at (87.5, 102.0)
- added U11: LPS25HB, Package_LGA:ST_HLGA-10_2.5x2.5mm_P0.6mm_LayoutBorder3x2y, B.Cu at (103.0, 74.9)
- BT1, BT2, C1, C12, C16, C17, C18, C19, C2, C20, J1, J2, J3, L1, M1, M2, N1, P1, Q1, Q2, Q3, R1, R10, R15, R24, R4, R5, R6, R9, SW1, U1, U2, U3, U4, U5, U7, U8, U9: moved to B.Cu
- U6: value LSM303A -> LSM303AGR; moved to B.Cu
- moved Q1 161.4 mm to (54.2, 95.0), turned to 270 degrees
- moved R3 159.8 mm to (48.0, 97.5), turned to 180 degrees
- moved R20 156.3 mm to (57.8, 94.0), turned to 270 degrees
- moved R24 152.3 mm to (60.9, 87.7), turned to 180 degrees
- moved C16 152.0 mm to (54.2, 87.6)
- moved U12 147.7 mm to (59.5, 100.0), turned to 90 degrees
- moved BT2 146.1 mm to (43.0, 101.8)
- moved C18 145.3 mm to (65.6, 74.0)
- moved LED2 144.2 mm to (70.5, 73.0), turned to 270 degrees
- moved R11 144.2 mm to (70.5, 76.5), turned to 90 degrees
- moved R23 143.4 mm to (64.0, 94.0), turned to 270 degrees
- moved R19 143.3 mm to (56.2, 94.0), turned to 270 degrees
- moved C19 142.2 mm to (68.2, 83.2)
- moved R13 141.2 mm to (68.5, 76.5), turned to 90 degrees
- moved R22 138.4 mm to (62.4, 94.0), turned to 270 degrees
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Connections:
- BT2 pad 2: +3V3 -> GND
- C1 pad 1: +3V3 -> GND
- C10 pad 2: +3V3 -> GND
- C11 pad 2: +3V3 -> GND
- C12 pad 2: +3V3 -> GND
- C13 pad 2: +3V3 -> GND
- C14 pad 2: +3V3 -> GND
- C15 pad 2: +3V3 -> GND
- C16 pad 2: +3V3 -> GND
- C17 pad 2: +3V3 -> GND
- C18 pad 2: +3V3 -> GND
- C19 pad 2: +3V3 -> GND
- C2 pad 2: +3V3 -> GND
- C20 pad 2: +3V3 -> GND
- C3 pad 2: +3V3 -> GND
- C4 pad 2: +3V3 -> GND
- C5 pad 2: +3V3 -> GND
- C6 pad 2: +3V3 -> GND
- C7 pad 2: +3V3 -> GND
- C8 pad 2: +3V3 -> GND
- C9 pad 2: +3V3 -> GND
- COM1 pad 20: +3V3 -> GND
- COM1 pad 28: +3V3 -> GND
- COM1 pad 30: +3V3 -> GND
- COM1 pad 31: +3V3 -> GND
- COM1 pad 32: +3V3 -> GND
- F1 pad 2: +3V3 -> GND
- J1 pad 2: +3V3 -> GND
- J2 pad 5: +3V3 -> GND
- J3 pad 5: +3V3 -> GND
- LED2 pad 1: +3V3 -> GND
- LED3 pad 1: +3V3 -> GND
- LED4 pad 1: +3V3 -> GND
- LED5 pad 1: +3V3 -> GND
- LED6 pad 1: +3V3 -> GND
- LED7 pad 1: +3V3 -> GND
- N1 pad 2: +3V3 -> GND
- P1 pad 4: +3V3 -> GND
- Q1 pad 2: Net-(Q1-Pad2) -> GND
- Q1 pad 4: +3V3 -> Net-(Q1-Pad4)
- Q1 pad 5: Net-(BT2-Pad1) -> Net-(Q1-Pad5)
- Q1 pad 6: Net-(BT2-Pad1) -> Net-(Q1-Pad5)
- Q1 pad 7: Net-(Q1-Pad7) -> Net-(BT2-Pad1)
- Q1 pad 8: Net-(Q1-Pad7) -> Net-(BT2-Pad1)
- Q3 pad 2: +3V3 -> GND
- R20 pad 2: Net-(R20-Pad2) -> +3V3
- R3 pad 2: Net-(Q1-Pad2) -> Net-(Q1-Pad4)
- R4 pad 1: Net-(Q1-Pad7) -> Net-(Q1-Pad5)
- SD1 pad 6: +3V3 -> GND
- SW1 pad 1: +3V3 -> GND
- SW1 pad 2: Net-(Q1-Pad2) -> Net-(Q1-Pad4)
- U1 pad 2: /Nichrome -> /LED_L0
- U1 pad 22: /LED_L0 -> /Nichrome
- U1 pad 23: +3V3 -> GND
- U1 pad 35: +3V3 -> GND
- U1 pad 44: +3V3 -> GND
- U1 pad 47: +3V3 -> GND
- U1 pad 8: +3V3 -> GND
- U10 pad 8: +3V3 -> GND
- U12 pad 8: +3V3 -> GND
- U2 pad 12: +3V3 -> GND
- U2 pad 18: +3V3 -> GND
- U2 pad 60: +3V3 -> GND
- U2 pad 63: +3V3 -> GND
- U3 pad 1: +3V3 -> GND
- U3 pad 10: Net-(Q1-Pad7) -> Net-(Q1-Pad5)
- U3 pad 2: +3V3 -> GND
- U3 pad 7: +3V3 -> GND
- U4 pad 1: +3V3 -> GND
- U4 pad 4: +3V3 -> GND
- U4 pad 5: +3V3 -> GND
- U4 pad 9: +3V3 -> GND
- U5 pad 4: +3V3 -> GND
- U6 pad 6: +3V3 -> GND
- U6 pad 8: +3V3 -> GND
- U7 pad 12: +3V3 -> GND
- U7 pad 2: +3V3 -> GND
- U7 pad 4: +3V3 -> GND
- U7 pad 5: +3V3 -> GND
- U8 pad 1: +3V3 -> GND
- U8 pad 10: +3V3 -> GND
- U8 pad 12: +3V3 -> GND
- U9 pad 1: +3V3 -> GND
- U9 pad 12: +3V3 -> GND
- U9 pad 3: +3V3 -> GND
- U9 pad 4: +3V3 -> GND
- U9 pad 6: +3V3 -> GND
Routing:
- net +3V3: track 0.00 -> 334.3 mm, vias 0 -> 18
- net +BATT: track 0.00 -> 152.8 mm, vias 0 -> 5
- net GND: track 0.00 -> 123.5 mm, vias 0 -> 60
- net /SDA: track 0.00 -> 104.2 mm, vias 0 -> 7
- net /SCL: track 0.00 -> 97.4 mm, vias 0 -> 10
- net Net-(BT2-Pad1): track 0.00 -> 73.9 mm, vias 0 -> 1
- net /MotorL_0: track 0.00 -> 71.8 mm, vias 0 -> 1
- net /MotorL_1: track 0.00 -> 71.4 mm, vias 0 -> 1
- net Net-(BT1-Pad1): track 0.00 -> 65.6 mm
- net /SUB_EN: track 0.00 -> 58.1 mm, vias 0 -> 2
- net /MAIN←SUB: track 0.00 -> 54.0 mm, vias 0 -> 2
- net /MAIN→SUB: track 0.00 -> 53.2 mm
- net +4V: track 0.00 -> 41.8 mm, vias 0 -> 3
- net /FlightPin: track 0.00 -> 41.7 mm
- net /TX_F: track 0.00 -> 35.2 mm, vias 0 -> 1
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- added copper zone on B.Cu, net GND
- added copper zone on F.Cu, net GND
Other:
- board size 4.3 x 3.1 mm -> 100 x 56 mm
- board text added: "+ -"
- board text added: "LightWeight CanSat Project for ARLISS 2020. 2019.10.18 Ver 1.0 Prototype (TRC16 EM) @n_yosihisa"
- board text added: "MAIN COM TX"
- board text added: "ON OFF"
- board text added: "PRG"
- board text added: "RST"
- board text added: "SUB PWR BATT"

Commit message: Update PCB
TRC16 EM1 発注
Parts:
- added C23: 0.1u, Capacitor_SMD:C_0603_1608Metric_Pad1.05x0.95mm_HandSolder, B.Cu at (75.5, 75.7)
- added G***: LOGO, CanSat2020_P:byakko_logo, F.Cu at (119.5, 84.0)
Connections:
- U1 pad 5: Net-(U1-Pad5) -> /IMG_MODE
- U2 pad 27: Net-(U2-Pad27) -> /IMG_MODE
Routing:
- net /IMG_MODE: track 0.00 -> 57.2 mm, vias 0 -> 2
- net GND: track 123.5 -> 132.1 mm, vias 60 -> 70
- net /MotorR_0: track 23.7 -> 22.2 mm
- net /FlightPin: track 41.7 -> 42.9 mm
Other:
- board text added: "LightWeight CanSat Project for ARLISS 2020. 2019.10.18 Ver 1.0 Prototype (TRC16 EM1) @n_yosihisa"
- board text added: "P TRC16 EM1"
- board text removed: "LightWeight CanSat Project for ARLISS 2020. 2019.10.18 Ver 1.0 Prototype (TRC16 EM) @n_yosihisa"
