File: PCB/CanSat2020_P/CanSat2020_P.sch (KiCad schematic (older format))
At the start: 82 parts, among them J1 GNSS Antenna, J2 Debug_L0, J3 Debug_F2, M1 Motor_L, M2 Motor_R, P1 C1098, Q1 FDS4935A, Q2 MTM231102LBF, Q3 2SC2712, SW1 POWER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

Commit message: Add LPS25HBTR
Parts:
- added C21, C22: 0.1u, Capacitor_SMD:C_0603_1608Metric_Pad1.05x0.95mm_HandSolder, symbol Device:C_Small
- added U11: LPS25HB, Package_LGA:ST_HLGA-10_2.5x2.5mm_P0.6mm_LayoutBorder3x2y, symbol Sensor_Pressure:LPS25HB
- U6: value LSM303A -> LSM303AGR
Connections:
- wire segments 411 -> 430
Other:
- note added: "R:0x53\nW:0x52"
- note added: "R:0x81\nW:0x80"
- note added: "R:0xA7\nW:0xA6"
- note added: "R:0xBB\nW:0xBA"
- note added: "XL\nR:0x33\nW:0x32\n\nMAG\nR:0x3D\nW:0x3C"

Commit message: Update PCB
Parts:
- added P2: Charge, Connector_JST:JST_EH_B03B-EH-A_1x03_P2.50mm_Vertical, symbol Connector_Generic:Conn_01x03
Connections:
- wire segments 430 -> 439
Changed lines of the file:
@@
 L user_library:FDS4935A Q1
 U 1 1 5DA5BC73
+P 2950 1200
+F 0 "Q1" V 3375 1200 50  0000 C CNN
+F 1 "FDS4935A" V 3284 1200 50  0000 C CNN
+F 2 "Package_SO:SOIC-8_3.9x4.9mm_P1.27mm" H 3150 1300 50  0001 C CNN
+F 3 "~" H 2950 1200 50  0001 C CNN
+F 4 "I-01246" H 700 0   50  0001 C CNN "秋月"
+	1    2950 1200
+	0    1    -1   0
+$EndComp
+$Comp
+L user_library:FDS4935A Q1
+U 2 1 5DA5BCB6
 P 2250 1200
 F 0 "Q1" V 2675 1200 50  0000 C CNN
@@
 F 2 "Package_SO:SOIC-8_3.9x4.9mm_P1.27mm" H 2450 1300 50  0001 C CNN
 F 3 "~" H 2250 1200 50  0001 C CNN
-F 4 "I-01246" H 0   0   50  0001 C CNN "秋月"
-	1    2250 1200
+F 4 "I-01246" H -700 0   50  0001 C CNN "秋月"
+	2    2250 1200
 	0    -1   -1   0
-$EndComp
-$Comp
-L user_library:FDS4935A Q1
-U 2 1 5DA5BCB6
-P 2950 1200
-F 0 "Q1" V 3375 1200 50  0000 C CNN
-F 1 "FDS4935A" V 3284 1200 50  0000 C CNN
-F 2 "Package_SO:SOIC-8_3.9x4.9mm_P1.27mm" H 3150 1300 50  0001 C CNN
-F 3 "~" H 2950 1200 50  0001 C CNN
-F 4 "I-01246" H 0   0   50  0001 C CNN "秋月"
-	2    2950 1200
-	0    1    -1   0
 $EndComp
 $Comp
@@
 $EndComp
 Wire Wire Line
-	1750 1100 2000 1100
+	1750 1100 1800 1100
 Wire Wire Line
 	2050 1000 2000 1000
@@
 Text Label 1450 3600 2    50   ~ 0
 FlightPin
+Text Label 1450 5000 2    50   ~ 0
+Nichrome
 Text Label 1450 3500 2    50   ~ 0
-Nichrome
-Text Label 1450 5000 2    50   ~ 0
 LED_L0
 Text Label 2950 9400 0    50   ~ 0
@@
 	1350 8000 1450 8000
 Wire Wire Line
-	1350 8800 1450 8800
-Wire Wire Line
 	1450 8900 1350 8900
 Wire Wire Line
@@
 Wire Wire Line
 	5750 8500 5750 9350
-Wire Wire Line
-	5200 8600 5200 8500
 Connection ~ 5200 8500
 Wire Wire Line
@@
 Text Notes 4850 2150 2    50   ~ 0
 R:0x81\nW:0x80
+$Comp
+L Connector_Generic:Conn_01x03 P2
+U 1 1 5DAB2B3F
+P 800 1950
+F 0 "P2" H 720 1625 50  0000 C CNN
+F 1 "Charge" H 720 1716 50  0000 C CNN
+F 2 "Connector_JST:JST_EH_B03B-EH-A_1x03_P2.50mm_Vertical" H 800 1950 50  0001 C CNN
+F 3 "~" H 800 1950 50  0001 C CNN
+	1    800  1950
+	-1   0    0    1
+$EndComp
+Wire Wire Line
+	1000 1850 1800 1850
+Wire Wire Line
+	1800 1850 1800 1100
+Wire Wire Line
+	1800 1100 2000 1100
+Connection ~ 1800 1100
+Wire Wire Line
+	750  1200 750  1500
+Wire Wire Line
+	750  1500 1150 1500
+Wire Wire Line
+	1150 1500 1150 1950
+Wire Wire Line
+	1150 1950 1000 1950
+Connection ~ 750  1200
+$Comp
+L power:GND #PWR0103
+U 1 1 5DB1BEFF
+P 1100 2100
+F 0 "#PWR0103" H 1100 1850 50  0001 C CNN
+F 1 "GND" H 1105 1927 50  0000 C CNN
+F 2 "" H 1100 2100 50  0001 C CNN
+F 3 "" H 1100 2100 50  0001 C CNN
+	1    1100 2100
+	1    0    0    -1
+$EndComp
+Wire Wire Line
+	1000 2050 1100 2050
+Wire Wire Line
+	1100 2050 1100 2100
+Wire Wire Line
+	5200 8500 5200 8650
+Wire Wire Line
+	1350 8800 1450 8800
 $EndSCHEMATC

Commit message: Add GS
Parts:
- U11: RS (none) -> 110-6550
Changed lines of the file:
@@
 F 2 "Package_LGA:ST_HLGA-10_2.5x2.5mm_P0.6mm_LayoutBorder3x2y" H 8950 7750 50  0001 C CNN
 F 3 "www.st.com/resource/en/datasheet/lps25hb.pdf" H 9000 7600 50  0001 C CNN
+F 4 "110-6550" H 0   0   50  0001 C CNN "RS"
 	1    8950 7950
 	-1   0    0    -1

Commit message: Update PCB
TRC16 EM1 発注
Parts:
- added C23: 0.1u, Capacitor_SMD:C_0603_1608Metric_Pad1.05x0.95mm_HandSolder, symbol Device:C_Small
Connections:
- net labels added: IMG_MODE
- wire segments 439 -> 442
Changed lines of the file:
@@
 FlightPin
 Wire Wire Line
-	11200 9200 11500 9200
+	11200 9200 11300 9200
 Wire Wire Line
 	11500 9200 11500 9150
@@
 Text Label 2950 9300 0    50   ~ 0
 MAIN←SUB
-Text Label 2950 8400 0    50   ~ 0
+Text Label 3000 8400 0    50   ~ 0
 SUB_EN
 Wire Wire Line
@@
 Wire Wire Line
 	1350 8800 1450 8800
+Text Label 1450 3200 2    50   ~ 0
+IMG_MODE
+Wire Wire Line
+	1450 3200 1550 3200
+Text Label 3000 8300 0    50   ~ 0
+IMG_MODE
+Wire Wire Line
+	3000 8300 2850 8300
+$Comp
+L Device:C_Small C23
+U 1 1 5DB474B6
+P 11300 9300
+F 0 "C23" H 11392 9346 50  0000 L CNN
+F 1 "0.1u" H 11392 9255 50  0000 L CNN
+F 2 "Capacitor_SMD:C_0603_1608Metric_Pad1.05x0.95mm_HandSolder" H 11300 9300 50  0001 C CNN
+F 3 "~" H 11300 9300 50  0001 C CNN
+	1    11300 9300
+	-1   0    0    -1
+$EndComp
+Connection ~ 11300 9200
+Wire Wire Line
+	11300 9200 11500 9200
+$Comp
+L power:GND #PWR0104
+U 1 1 5DB47915
+P 11300 9400
+F 0 "#PWR0104" H 11300 9150 50  0001 C CNN
+F 1 "GND" H 11305 9227 50  0000 C CNN
+F 2 "" H 11300 9400 50  0001 C CNN
+F 3 "" H 11300 9400 50  0001 C CNN
+	1    11300 9400
+	1    0    0    -1
+$EndComp
 $EndSCHEMATC
